Commit message: Began building body

File: body.urdf (robot description, URDF)
Before this commit: robot robot, 9 links, 8 joints
Links:
- removed link LeftLeg
- removed link LeftLowerLeg
- removed link RightLeg
- removed link RightLowerLeg
- link BackLeg: geometry collision box size=0.2 0.2 0.2; visual box size=0.2 0.2 0.2
- link BackLowerLeg: geometry collision box size=0.2 0.25 1; visual box size=0.2 0.25 1
- link FrontLeg: geometry collision box size=0.2 0.2 0.2; visual box size=0.2 0.2 0.2
- link FrontLowerLeg: geometry collision box size=0.2 0.25 1; visual box size=0.2 0.25 1
- link Torso: geometry collision box size=1 1 1.5; visual box size=1 1 1.5
Joints:
- removed joint LeftLeg_LeftLowerLeg
- removed joint RightLeg_RightLowerLeg
- removed joint Torso_LeftLeg
- removed joint Torso_RightLeg
- joint BackLeg_BackLowerLeg: origin xyz=0 -1 0 rpy=0 0 0 -> xyz=0 -0.5 0 rpy=0 0 0
- joint FrontLeg_FrontLowerLeg: origin xyz=0 1 0 rpy=0 0 0 -> xyz=0 0.5 0 rpy=0 0 0
- joint Torso_BackLeg: origin xyz=0 -0.5 1 rpy=0 0 0 -> xyz=0 -0.2 1 rpy=0 0 0
- joint Torso_FrontLeg: origin xyz=0 0.5 1 rpy=0 0 0 -> xyz=0 0.2 1 rpy=0 0 0

Commit message: Changed variable names

File: body.urdf (robot description, URDF)
Before this commit: robot robot, 11 links, 10 joints
Links:
- removed link BackLeg
- removed link BackLowerLeg
- removed link FrontLeg
- removed link FrontLowerLeg
- removed link LeftLeg
- removed link LeftLowerLeg
- removed link RightLeg
- removed link RightLowerLeg
- added link ArmOne, mass 1; collision box size=0.2 0.25 0.75; visual box size=0.2 0.25 0.75
- added link ArmTwo, mass 1; collision box size=0.2 0.25 0.75; visual box size=0.2 0.25 0.75
- added link LowerLegOne, mass 1; collision box size=0.2 0.2 0.4; visual box size=0.2 0.2 0.4
- added link LowerLegTwo, mass 1; collision box size=0.2 0.2 0.4; visual box size=0.2 0.2 0.4
- added link ShoulderOne, mass 1; collision box size=0.2 0.2 0.2; visual box size=0.2 0.2 0.2
- added link ShoulderTwo, mass 1; collision box size=0.2 0.2 0.2; visual box size=0.2 0.2 0.2
- added link UpperLegOne, mass 1; collision box size=0.2 0.2 0.5; visual box size=0.2 0.2 0.5
- added link UpperLegTwo, mass 1; collision box size=0.2 0.2 0.5; visual box size=0.2 0.2 0.5
Joints:
- removed joint BackLeg_BackLowerLeg
- removed joint FrontLeg_FrontLowerLeg
- removed joint LeftLeg_LeftLowerLeg
- removed joint LeftLowerLeg_FootOne
- removed joint RightLeg_RightLowerLeg
- removed joint RightLowerLeg_FootTwo
- removed joint Torso_BackLeg
- removed joint Torso_FrontLeg
- removed joint Torso_LeftLeg
- removed joint Torso_RightLeg
- added joint LowerLegOne_FootOne: type revolute, parent LowerLegOne, child FootOne, origin xyz=0 0 -0.4 rpy=0 0 0, axis 0 1 0, limit lower=-3.14159 upper=3.14159 effort=0.0 velocity=0.0
- added joint LowerLegTwo_FootTwo: type revolute, parent LowerLegTwo, child FootTwo, origin xyz=0 0 -0.4 rpy=0 0 0, axis 0 1 0, limit lower=-3.14159 upper=3.14159 effort=0.0 velocity=0.0
- added joint ShoulderOne_ArmTwo: type revolute, parent ShoulderOne, child ArmTwo, origin xyz=0 0.2 -0.1 rpy=0 0 0, axis 1 0 0, limit lower=-3.14159 upper=3.14159 effort=0.0 velocity=0.0
- added joint ShoulderTwo_ArmOne: type revolute, parent ShoulderTwo, child ArmOne, origin xyz=0 -0.2 -0.1 rpy=0 0 0, axis 1 0 0, limit lower=-3.14159 upper=3.14159 effort=0.0 velocity=0.0
- added joint Torso_ShoulderOne: type revolute, parent Torso, child ShoulderOne, origin xyz=0 1.25 2.2 rpy=0 0 0, axis 0 1 0, limit lower=-3.14159 upper=3.14159 effort=0.0 velocity=0.0
- added joint Torso_ShoulderTwo: type revolute, parent Torso, child ShoulderTwo, origin xyz=0 0.75 2.2 rpy=0 0 0, axis 0 1 0, limit lower=-3.14159 upper=3.14159 effort=0.0 velocity=0.0
- added joint Torso_UpperLegOne: type revolute, parent Torso, child UpperLegOne, origin xyz=0 0.875 1.5 rpy=0 0 0, axis 0 1 0, limit lower=-3.14159 upper=3.14159 effort=0.0 velocity=0.0
- added joint Torso_UpperLegTwo: type revolute, parent Torso, child UpperLegTwo, origin xyz=0 1.125 1.5 rpy=0 0 0, axis 0 1 0, limit lower=-3.14159 upper=3.14159 effort=0.0 velocity=0.0
- added joint UpperLegOne_LowerLegOne: type revolute, parent UpperLegOne, child LowerLegOne, origin xyz=0 0 -0.5 rpy=0 0 0, axis 0 1 0, limit lower=-3.14159 upper=3.14159 effort=0.0 velocity=0.0
- added joint UpperLegTwo_LowerLegTwo: type revolute, parent UpperLegTwo, child LowerLegTwo, origin xyz=0 0 -0.5 rpy=0 0 0, axis 0 1 0, limit lower=-3.14159 upper=3.14159 effort=0.0 velocity=0.0

Commit message: Final push

File: body.urdf (robot description, URDF)
Before this commit: robot robot, 11 links, 10 joints
Links:
- link ArmOne: geometry collision box size=0.2 0.2 0.75; visual box size=0.2 0.2 0.75
- link ArmTwo: geometry collision box size=0.2 0.2 0.75; visual box size=0.2 0.2 0.75
Joints:
- joint LowerLegOne_FootOne: limit lower=-3.14159 upper=3.14159 effort=0.0 velocity=0.0 -> lower=-0.2617993877991494 upper=0.2617993877991494 effort=0.0 velocity=0.0
- joint LowerLegTwo_FootTwo: limit lower=-3.14159 upper=3.14159 effort=0.0 velocity=0.0 -> lower=-0.2617993877991494 upper=0.2617993877991494 effort=0.0 velocity=0.0
- joint ShoulderOne_ArmTwo: limit lower=-3.14159 upper=3.14159 effort=0.0 velocity=0.0 -> lower=-3.141592653589793 upper=3.141592653589793 effort=0.0 velocity=0.0
- joint ShoulderTwo_ArmOne: limit lower=-3.14159 upper=3.14159 effort=0.0 velocity=0.0 -> lower=-3.141592653589793 upper=3.141592653589793 effort=0.0 velocity=0.0
- joint Torso_ShoulderOne: limit lower=-3.14159 upper=3.14159 effort=0.0 velocity=0.0 -> lower=-3.141592653589793 upper=3.141592653589793 effort=0.0 velocity=0.0
- joint Torso_ShoulderTwo: limit lower=-3.14159 upper=3.14159 effort=0.0 velocity=0.0 -> lower=-3.141592653589793 upper=3.141592653589793 effort=0.0 velocity=0.0
- joint Torso_UpperLegOne: limit lower=-3.14159 upper=3.14159 effort=0.0 velocity=0.0 -> lower=-0.7853981633974483 upper=0.7853981633974483 effort=0.0 velocity=0.0
- joint Torso_UpperLegTwo: limit lower=-3.14159 upper=3.14159 effort=0.0 velocity=0.0 -> lower=-0.7853981633974483 upper=0.7853981633974483 effort=0.0 velocity=0.0
- joint UpperLegOne_LowerLegOne: limit lower=-3.14159 upper=3.14159 effort=0.0 velocity=0.0 -> lower=0 upper=0.2617993877991494 effort=0.0 velocity=0.0
- joint UpperLegTwo_LowerLegTwo: limit lower=-3.14159 upper=3.14159 effort=0.0 velocity=0.0 -> lower=0 upper=0.2617993877991494 effort=0.0 velocity=0.0

Commit message: Finished many legs

File: body.urdf (robot description, URDF)
Before this commit: robot robot, 9 links, 8 joints
Links:
- added link BackLegTwo, mass 1; collision box size=0.2 1 0.2; visual box size=0.2 1 0.2
- added link BackLowerLegTwo, mass 1; collision box size=0.2 0.2 1; visual box size=0.2 0.2 1
- added link FrontLegTwo, mass 1; collision box size=0.2 1 0.2; visual box size=0.2 1 0.2
- added link FrontLowerLegTwo, mass 1; collision box size=0.2 0.2 1; visual box size=0.2 0.2 1
- added link LeftLegTwo, mass 1; collision box size=1 0.2 0.2; visual box size=1 0.2 0.2
- added link LeftLowerLegTwo, mass 1; collision box size=0.2 0.2 1; visual box size=0.2 0.2 1
- added link RightLegTwo, mass 1; collision box size=1 0.2 0.2; visual box size=1 0.2 0.2
- added link RightLowerLegTwo, mass 1; collision box size=0.2 0.2 1; visual box size=0.2 0.2 1
Joints:
- added joint BackLegTwo_BackLowerLegTwo: type revolute, parent BackLegTwo, child BackLowerLegTwo, origin xyz=0 -1 0 rpy=0 0 0, axis 1 0 0, limit lower=-3.14159 upper=3.14159 effort=0.0 velocity=0.0
- added joint FrontLegTwo_FrontLowerLegTwo: type revolute, parent FrontLegTwo, child FrontLowerLegTwo, origin xyz=0 1 0 rpy=0 0 0, axis 1 0 0, limit lower=-3.14159 upper=3.14159 effort=0.0 velocity=0.0
- added joint LeftLegTwo_LeftLowerLegTwo: type revolute, parent LeftLegTwo, child LeftLowerLegTwo, origin xyz=-1 0 0 rpy=0 0 0, axis 0 1 0, limit lower=-3.14159 upper=3.14159 effort=0.0 velocity=0.0
- added joint RightLegTwo_RightLowerLegTwo: type revolute, parent RightLegTwo, child RightLowerLegTwo, origin xyz=1 0 0 rpy=0 0 0, axis 0 1 0, limit lower=-3.14159 upper=3.14159 effort=0.0 velocity=0.0
- added joint Torso_BackLegTwo: type revolute, parent Torso, child BackLegTwo, origin xyz=0.25 -0.5 1 rpy=0 0 0, axis 1 0 0, limit lower=-3.14159 upper=3.14159 effort=0.0 velocity=0.0
- added joint Torso_FrontLegTwo: type revolute, parent Torso, child FrontLegTwo, origin xyz=-0.25 0.5 1 rpy=0 0 0, axis 1 0 0, limit lower=-3.14159 upper=3.14159 effort=0.0 velocity=0.0
- added joint Torso_LeftLegTwo: type revolute, parent Torso, child LeftLegTwo, origin xyz=-0.5 -0.25 1 rpy=0 0 0, axis 0 1 0, limit lower=-3.14159 upper=3.14159 effort=0.0 velocity=0.0
- added joint Torso_RightLegTwo: type revolute, parent Torso, child RightLegTwo, origin xyz=0.5 -0.25 1 rpy=0 0 0, axis 0 1 0, limit lower=-3.14159 upper=3.14159 effort=0.0 velocity=0.0
- joint Torso_BackLeg: origin xyz=0 -0.5 1 rpy=0 0 0 -> xyz=-0.25 -0.5 1 rpy=0 0 0
- joint Torso_FrontLeg: origin xyz=0 0.5 1 rpy=0 0 0 -> xyz=0.25 0.5 1 rpy=0 0 0
- joint Torso_LeftLeg: origin xyz=-0.5 0 1 rpy=0 0 0 -> xyz=-0.5 0.25 1 rpy=0 0 0
- joint Torso_RightLeg: origin xyz=0.5 0 1 rpy=0 0 0 -> xyz=0.5 0.25 1 rpy=0 0 0

Commit message: Built platform

File: body.urdf (robot description, URDF)
Before this commit: robot robot, 9 links, 8 joints
Joints:
- joint Torso_BackLeg: origin xyz=0 -0.5 1 rpy=0 0 0 -> xyz=0 -0.5 4 rpy=0 0 0
- joint Torso_FrontLeg: origin xyz=0 0.5 1 rpy=0 0 0 -> xyz=0 0.5 4 rpy=0 0 0
- joint Torso_LeftLeg: origin xyz=-0.5 0 1 rpy=0 0 0 -> xyz=-0.5 0 4 rpy=0 0 0
- joint Torso_RightLeg: origin xyz=0.5 0 1 rpy=0 0 0 -> xyz=0.5 0 4 rpy=0 0 0

Commit message: Finished runway

File: body.urdf (robot description, URDF)
Before this commit: robot robot, 9 links, 8 joints
Joints:
- joint Torso_BackLeg: origin xyz=0 -0.5 4 rpy=0 0 0 -> xyz=0 -0.5 3 rpy=0 0 0
- joint Torso_FrontLeg: origin xyz=0 0.5 4 rpy=0 0 0 -> xyz=0 0.5 3 rpy=0 0 0
- joint Torso_LeftLeg: origin xyz=-0.5 0 4 rpy=0 0 0 -> xyz=-0.5 0 3 rpy=0 0 0
- joint Torso_RightLeg: origin xyz=0.5 0 4 rpy=0 0 0 -> xyz=0.5 0 3 rpy=0 0 0
